Commit message: 更新urdf

File: src/lycus_moveit_config/config/lycus.ros2_control.xacro (robot description, xacro)
@@ -7,169 +7,169 @@
                 <plugin>mock_components/GenericSystem</plugin>
             </hardware>
-            <joint name="AR5-5_08L-W4C1C9-ZY2_joint_1">
+            <joint name="AR5-5_08L-W4C1C5-ZY2_joint_1">
                 <command_interface name="position"/>
                 <state_interface name="position">
-                  <param name="initial_value">${initial_positions['AR5-5_08L-W4C1C9-ZY2_joint_1']}</param>
+                  <param name="initial_value">${initial_positions['AR5-5_08L-W4C1C5-ZY2_joint_1']}</param>
                 </state_interface>
                 <state_interface name="velocity"/>
             </joint>
-            <joint name="AR5-5_08L-W4C1C9-ZY2_joint_2">
+            <joint name="AR5-5_08L-W4C1C5-ZY2_joint_2">
                 <command_interface name="position"/>
                 <state_interface name="position">
-                  <param name="initial_value">${initial_positions['AR5-5_08L-W4C1C9-ZY2_joint_2']}</param>
+                  <param name="initial_value">${initial_positions['AR5-5_08L-W4C1C5-ZY2_joint_2']}</param>
                 </state_interface>
                 <state_interface name="velocity"/>
             </joint>
-            <joint name="AR5-5_08L-W4C1C9-ZY2_joint_3">
+            <joint name="AR5-5_08L-W4C1C5-ZY2_joint_3">
                 <command_interface name="position"/>
                 <state_interface name="position">
-                  <param name="initial_value">${initial_positions['AR5-5_08L-W4C1C9-ZY2_joint_3']}</param>
+                  <param name="initial_value">${initial_positions['AR5-5_08L-W4C1C5-ZY2_joint_3']}</param>
                 </state_interface>
                 <state_interface name="velocity"/>
             </joint>
-            <joint name="AR5-5_08L-W4C1C9-ZY2_joint_4">
+            <joint name="AR5-5_08L-W4C1C5-ZY2_joint_4">
                 <command_interface name="position"/>
                 <state_interface name="position">
-                  <param name="initial_value">${initial_positions['AR5-5_08L-W4C1C9-ZY2_joint_4']}</param>
+                  <param name="initial_value">${initial_positions['AR5-5_08L-W4C1C5-ZY2_joint_4']}</param>
                 </state_interface>
                 <state_interface name="velocity"/>
             </joint>
-            <joint name="AR5-5_08L-W4C1C9-ZY2_joint_5">
+            <joint name="AR5-5_08L-W4C1C5-ZY2_joint_5">
                 <command_interface name="position"/>
                 <state_interface name="position">
-                  <param name="initial_value">${initial_positions['AR5-5_08L-W4C1C9-ZY2_joint_5']}</param>
+                  <param name="initial_value">${initial_positions['AR5-5_08L-W4C1C5-ZY2_joint_5']}</param>
                 </state_interface>
                 <state_interface name="velocity"/>
             </joint>
-            <joint name="AR5-5_08L-W4C1C9-ZY2_joint_6">
+            <joint name="AR5-5_08L-W4C1C5-ZY2_joint_6">
                 <command_interface name="position"/>
                 <state_interface name="position">
-                  <param name="initial_value">${initial_positions['AR5-5_08L-W4C1C9-ZY2_joint_6']}</param>
+                  <param name="initial_value">${initial_positions['AR5-5_08L-W4C1C5-ZY2_joint_6']}</param>
                 </state_interface>
                 <state_interface name="velocity"/>
             </joint>
-            <joint name="AR5-5_08L-W4C1C9-ZY2_joint_7">
+            <joint name="AR5-5_08L-W4C1C5-ZY2_joint_7">
                 <command_interface name="position"/>
                 <state_interface name="position">
-                  <param name="initial_value">${initial_positions['AR5-5_08L-W4C1C9-ZY2_joint_7']}</param>
+                  <param name="initial_value">${initial_positions['AR5-5_08L-W4C1C5-ZY2_joint_7']}</param>
                 </state_interface>
                 <state_interface name="velocity"/>
             </joint>
-            <joint name="AR5-5_08R-W4C1C9-ZY2_joint_1">
+            <joint name="AR5-5_08R-W4C1C5-ZY2_joint_1">
                 <command_interface name="position"/>
                 <state_interface name="position">
-                  <param name="initial_value">${initial_positions['AR5-5_08R-W4C1C9-ZY2_joint_1']}</param>
+                  <param name="initial_value">${initial_positions['AR5-5_08R-W4C1C5-ZY2_joint_1']}</param>
                 </state_interface>
                 <state_interface name="velocity"/>
             </joint>
-            <joint name="AR5-5_08R-W4C1C9-ZY2_joint_2">
+            <joint name="AR5-5_08R-W4C1C5-ZY2_joint_2">
                 <command_interface name="position"/>
                 <state_interface name="position">
-                  <param name="initial_value">${initial_positions['AR5-5_08R-W4C1C9-ZY2_joint_2']}</param>
+                  <param name="initial_value">${initial_positions['AR5-5_08R-W4C1C5-ZY2_joint_2']}</param>
                 </state_interface>
                 <state_interface name="velocity"/>
             </joint>
-            <joint name="AR5-5_08R-W4C1C9-ZY2_joint_3">
+            <joint name="AR5-5_08R-W4C1C5-ZY2_joint_3">
                 <command_interface name="position"/>
                 <state_interface name="position">
-                  <param name="initial_value">${initial_positions['AR5-5_08R-W4C1C9-ZY2_joint_3']}</param>
+                  <param name="initial_value">${initial_positions['AR5-5_08R-W4C1C5-ZY2_joint_3']}</param>
                 </state_interface>
                 <state_interface name="velocity"/>
             </joint>
-            <joint name="AR5-5_08R-W4C1C9-ZY2_joint_4">
+            <joint name="AR5-5_08R-W4C1C5-ZY2_joint_4">
                 <command_interface name="position"/>
                 <state_interface name="position">
-                  <param name="initial_value">${initial_positions['AR5-5_08R-W4C1C9-ZY2_joint_4']}</param>
+                  <param name="initial_value">${initial_positions['AR5-5_08R-W4C1C5-ZY2_joint_4']}</param>
                 </state_interface>
                 <state_interface name="velocity"/>
             </joint>
-            <joint name="AR5-5_08R-W4C1C9-ZY2_joint_5">
+            <joint name="AR5-5_08R-W4C1C5-ZY2_joint_5">
                 <command_interface name="position"/>
                 <state_interface name="position">
-                  <param name="initial_value">${initial_positions['AR5-5_08R-W4C1C9-ZY2_joint_5']}</param>
+                  <param name="initial_value">${initial_positions['AR5-5_08R-W4C1C5-ZY2_joint_5']}</param>
                 </state_interface>
                 <state_interface name="velocity"/>
             </joint>
-            <joint name="AR5-5_08R-W4C1C9-ZY2_joint_6">
+            <joint name="AR5-5_08R-W4C1C5-ZY2_joint_6">
                 <command_interface name="position"/>
                 <state_interface name="position">
-                  <param name="initial_value">${initial_positions['AR5-5_08R-W4C1C9-ZY2_joint_6']}</param>
+                  <param name="initial_value">${initial_positions['AR5-5_08R-W4C1C5-ZY2_joint_6']}</param>
                 </state_interface>
                 <state_interface name="velocity"/>
             </joint>
-            <joint name="AR5-5_08R-W4C1C9-ZY2_joint_7">
+            <joint name="AR5-5_08R-W4C1C5-ZY2_joint_7">
                 <command_interface name="position"/>
                 <state_interface name="position">
-                  <param name="initial_value">${initial_positions['AR5-5_08R-W4C1C9-ZY2_joint_7']}</param>
+                  <param name="initial_value">${initial_positions['AR5-5_08R-W4C1C5-ZY2_joint_7']}</param>
                 </state_interface>
                 <state_interface name="velocity"/>
             </joint>
-            <joint name="Calf-joint">
+            <joint name="Calf_joint">
                 <command_interface name="position"/>
                 <state_interface name="position">
-                  <param name="initial_value">${initial_positions['Calf-joint']}</param>
+                  <param name="initial_value">${initial_positions['Calf_joint']}</param>
                 </state_interface>
                 <state_interface name="velocity"/>
             </joint>
-            <joint name="Thigh-joint">
+            <joint name="Thigh_joint">
                 <command_interface name="position"/>
                 <state_interface name="position">
-                  <param name="initial_value">${initial_positions['Thigh-joint']}</param>
+                  <param name="initial_value">${initial_positions['Thigh_joint']}</param>
                 </state_interface>
                 <state_interface name="velocity"/>
             </joint>
-            <joint name="Waist-joint">
+            <joint name="Waist_joint">
                 <command_interface name="position"/>
                 <state_interface name="position">
-                  <param name="initial_value">${initial_positions['Waist-joint']}</param>
+                  <param name="initial_value">${initial_positions['Waist_joint']}</param>
                 </state_interface>
                 <state_interface name="velocity"/>
             </joint>
-            <joint name="Chest-joint">
+            <joint name="Chest_joint">
                 <command_interface name="position"/>
                 <state_interface name="position">
-                  <param name="initial_value">${initial_positions['Chest-joint']}</param>
+                  <param name="initial_value">${initial_positions['Chest_joint']}</param>
                 </state_interface>
                 <state_interface name="velocity"/>
             </joint>
-            <joint name="Neck-joint">
+            <joint name="Neck_joint">
                 <command_interface name="position"/>
                 <state_interface name="position">
-                  <param name="initial_value">${initial_positions['Neck-joint']}</param>
+                  <param name="initial_value">${initial_positions['Neck_joint']}</param>
                 </state_interface>
                 <state_interface name="velocity"/>
             </joint>
-            <joint name="Head-joint">
+            <joint name="Head_joint">
                 <command_interface name="position"/>
                 <state_interface name="position">
-                  <param name="initial_value">${initial_positions['Head-joint']}</param>
+                  <param name="initial_value">${initial_positions['Head_joint']}</param>
                 </state_interface>
                 <state_interface name="velocity"/>
             </joint>
-            <joint name="Whee1-joint">
+            <joint name="Wheel1_joint">
                 <command_interface name="position"/>
                 <state_interface name="position">
-                  <param name="initial_value">${initial_positions['Whee1-joint']}</param>
+                  <param name="initial_value">${initial_positions['Wheel1_joint']}</param>
                 </state_interface>
                 <state_interface name="velocity"/>
             </joint>
-            <joint name="Whee2-joint">
+            <joint name="Wheel2_joint">
                 <command_interface name="position"/>
                 <state_interface name="position">
-                  <param name="initial_value">${initial_positions['Whee2-joint']}</param>
+                  <param name="initial_value">${initial_positions['Wheel2_joint']}</param>
                 </state_interface>
                 <state_interface name="velocity"/>
             </joint>
-            <joint name="Whee3-joint">
+            <joint name="Wheel3_joint">
                 <command_interface name="position"/>
                 <state_interface name="position">
-                  <param name="initial_value">${initial_positions['Whee3-joint']}</param>
+                  <param name="initial_value">${initial_positions['Wheel3_joint']}</param>
                 </state_interface>
                 <state_interface name="velocity"/>
             </joint>
-            <joint name="Whee4-joint">
+            <joint name="Wheel4_joint">
                 <command_interface name="position"/>
                 <state_interface name="position">
-                  <param name="initial_value">${initial_positions['Whee4-joint']}</param>
+                  <param name="initial_value">${initial_positions['Wheel4_joint']}</param>
                 </state_interface>
                 <state_interface name="velocity"/>

Commit message: 更新urdf添加夹爪stl模型

File: src/lycus_description/urdf/lycus.urdf (robot description, URDF)
Before this commit: robot lycus, 39 links, 38 joints
Links:
- added link left_gripper_base, mass 1.5; collision mesh filename=package://lycus_description/meshes/gripper_drive_motor.stl; visual mesh filename=package://lycus_description/meshes/gripper_drive_motor.stl
- added link left_gripper_left_jaw, mass 0.37669144; collision mesh filename=package://lycus_description/meshes/gripper_left_finger.stl; visual mesh filename=package://lycus_description/meshes/gripper_left_finger.stl
- added link left_gripper_right_jaw, mass 0.37669236; collision mesh filename=package://lycus_description/meshes/gripper_right_finger.stl; visual mesh filename=package://lycus_description/meshes/gripper_right_finger.stl
- added link right_gripper_base, mass 1.5; collision mesh filename=package://lycus_description/meshes/gripper_drive_motor.stl; visual mesh filename=package://lycus_description/meshes/gripper_drive_motor.stl
- added link right_gripper_left_jaw, mass 0.37669144; collision mesh filename=package://lycus_description/meshes/gripper_left_finger.stl; visual mesh filename=package://lycus_description/meshes/gripper_left_finger.stl
- added link right_gripper_right_jaw, mass 0.37669236; collision mesh filename=package://lycus_description/meshes/gripper_right_finger.stl; visual mesh filename=package://lycus_description/meshes/gripper_right_finger.stl
Joints:
- added joint left_gripper: type prismatic, parent left_gripper_base, child left_gripper_right_jaw, origin xyz=0.01 0.1675 0.00072458 rpy=0 0 0, axis 1 0 0, limit lower=-0.042 upper=0 effort=10 velocity=3
- added joint left_gripper_mimic: type prismatic, parent left_gripper_base, child left_gripper_left_jaw, origin xyz=-0.01 0.1675 -0.02877542 rpy=0 0 0, axis 1 0 0, limit lower=0 upper=0.042 effort=10 velocity=3, mimic joint=left_gripper multiplier=-1 offset=0
- added joint left_gripper_mount: type fixed, parent AR5-5_08L-W4C1C5-ZY2_flan_link, child left_gripper_base, origin xyz=0 0 0 rpy=1.5707963267948966 0 3.141592653589793
- added joint right_gripper: type prismatic, parent right_gripper_base, child right_gripper_right_jaw, origin xyz=0.01 0.1675 0.00072458 rpy=0 0 0, axis 1 0 0, limit lower=-0.042 upper=0 effort=10 velocity=3
- added joint right_gripper_mimic: type prismatic, parent right_gripper_base, child right_gripper_left_jaw, origin xyz=-0.01 0.1675 -0.02877542 rpy=0 0 0, axis 1 0 0, limit lower=0 upper=0.042 effort=10 velocity=3, mimic joint=right_gripper multiplier=-1 offset=0
- added joint right_gripper_mount: type fixed, parent AR5-5_08R-W4C1C5-ZY2_flan_link, child right_gripper_base, origin xyz=0 0 0 rpy=1.5707963267948966 0 0
- joint left_arm_ee_joint: origin xyz=0 0 0 rpy=1.5707963267948966 0 0 -> xyz=0 0.2465 0.011975 rpy=0 0 0; parent AR5-5_08L-W4C1C5-ZY2_flan_link -> left_gripper_base
- joint right_arm_ee_joint: origin xyz=0 0 0 rpy=1.5707963267948966 0 0 -> xyz=0 0.2465 0.011975 rpy=0 0 0; parent AR5-5_08R-W4C1C5-ZY2_flan_link -> right_gripper_base
