Commit message: 更新夹爪状态发布

File: src/lycus_moveit_config/config/lycus.ros2_control.xacro (robot description, xacro)
@@ -175,4 +175,17 @@
                 <state_interface name="velocity"/>
             </joint>
+            <!-- 只发布开合，不接入轨迹控制器。mimic 关节由 robot_state_publisher 计算。 -->
+            <joint name="left_gripper">
+                <state_interface name="position">
+                  <param name="initial_value">${initial_positions['left_gripper']}</param>
+                </state_interface>
+                <state_interface name="velocity"/>
+            </joint>
+            <joint name="right_gripper">
+                <state_interface name="position">
+                  <param name="initial_value">${initial_positions['right_gripper']}</param>
+                </state_interface>
+                <state_interface name="velocity"/>
+            </joint>
         </ros2_control>
     </xacro:macro>
